File: panel-box/board/panel-box.kicad_sch (KiCad schematic)
At the start: 6 parts, among them U1 ATSAMD11D14A-SS, X1 SWD

Commit message: WIP
Parts:
- added C?: 500u/100V, symbol Device:C_Polarized
- added C?: 1u/500V, symbol Device:C
- added F? (x2): Fuse, symbol Device:Fuse
- added J? (x2): Panel, symbol Connector:Conn_01x02_Female
Connections:
- net GND: now also C?.2, J?.1 (Pin_1), J?.1 (Pin_1)
- new net: F?.1, J?.2 (Pin_2) (x2)
- new net VIN: C?.1, F?.2
- new net VOUT: F?.2
- new net VOUT+: C?.1
- new net VOUT-: C?.2
Other:
- added sheet Flyback channel (flyback.kicad_sch)
- added sheet Flyback channel1 (flyback.kicad_sch)
- added sheet Flyback channel2 (flyback.kicad_sch)
- note added: "Konektor VIN - jaky? Konektor VOUT - jaky? - kolik? Konektor DATA - kolik? - pinout? DATA bus driver - jaky? - pullup? LDO 12V - jaky? LDO 3V3 - jaky? Mereni napeti VIN - jak? Mereni proudu VIN - jak? Mereni vystupniho napeti () - jak? - dioda? - napajeni izol. OPAMP? SYNC vstupni prizpusobeni - jak? NRST vstupni prizpusobeni - jak? Master I2C, EEPROM - pullup - vybrat EEPROM"
- moved on the sheet: D1, R1

Commit message: WIP
Connections:
- net PWM_Q1: no longer U1.20 (PA04)
- net PWM_Q2: no longer U1.1 (PA05)
- net PWM_Q3: no longer U1.2 (PA06)
- net SDA_MASTER: no longer names the net of U1.10 (PA23)
- net SDA_MASTER: no longer U1.9 (PA22)
- new net PWM_H1: U1.20 (PA04)
- new net PWM_H2: U1.1 (PA05)
- no-connect marks 3 -> 6
