File: board/optimizer.kicad_sch (KiCad schematic)
At the start: 45 parts

Commit message: WIP
Parts:
- removed C: C, symbol Device:C
- added C (x8): C, symbol Device:C
- added D: LED, symbol Device:LED
- added J: Conn_01x04_Female, symbol Connector:Conn_01x04_Female
- added R (x3): R, symbol Device:R
- added TP (x2): TestPoint_Probe, symbol Connector:TestPoint_Probe
- added U: MCP1416, Package_TO_SOT_SMD:SOT-23-5, symbol Driver_FET:MCP1416
Connections:
- net +12V: now also C.1, C.1, U.2 (Vdd)
- net +3V3: now also C.1, C.1, C.1, C.1, C.2, C.2, J.4 (Pin_4)
- net GND: now also C.1, C.1, C.2, C.2, C.2, C.2, C.2, C.2, D.1 (K), J.1 (Pin_1), U.4 (GND)
- net SWP_HI_PWM: now also U.10 (PA25)
- net SWP_HI_SEN: now also U.14 (PA04)
- net SWP_LO_PWM: now also U.9 (PA24)
- net SWP_LO_SEN: now also U.13 (PA02)
- net U_SEN: now also U.1 (PA05), R.2; no longer R.1
- net LED: now reaches U.2 (PA08/XIN)
- net LED: now also R.1
- net TEL1: now reaches U.4 (PA14)
- net TEL1: now also J.2 (Pin_2)
- net TEL2: now reaches U.5 (PA15)
- net TEL2: now also J.3 (Pin_3)
- net at U.2, U.7: now also TP.1, U.3 (IN)
- net GATE: no longer names the net of Q.1 (G)
- net GATE: now also TP.1, U.5 (OUT)
- new net: D.2 (A), R.2
- new net: R.1, R.1
- new net: R.1, R.2
- no-connect marks 0 -> 1
Other:
- moved on the sheet: C, R, U, UA, X
