File: board/optimizer.kicad_sch (KiCad schematic)
At the start: 60 parts

Commit message: WIP
Parts:
- added NT: NetTie_3_Tee, symbol Device:NetTie_3_Tee
Connections:
- new net: D.1 (K), L.1, NT.2
- new net: C.1, NT.1, NT.1
- new net: NT.3, R.2
Changed lines of the file:
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@@
   (junction (at 139.7 101.6) (diameter 0) (color 0 0 0 0)
   )
-  (junction (at 62.23 81.28) (diameter 0) (color 0 0 0 0)
+  (junction (at 55.88 81.28) (diameter 0) (color 0 0 0 0)
+  )
+  (junction (at 116.84 81.28) (diameter 0) (color 0 0 0 0)
+  )
+  (junction (at 128.27 132.08) (diameter 0) (color 0 0 0 0)
+  )
+  (junction (at 118.11 160.02) (diameter 0) (color 0 0 0 0)
+  )
+  (junction (at 60.96 134.62) (diameter 0) (color 0 0 0 0)
+  )
+  (junction (at 71.12 162.56) (diameter 0) (color 0 0 0 0)
+  )
+  (junction (at 106.68 91.44) (diameter 0) (color 0 0 0 0)
+  )
+  (junction (at 134.62 158.75) (diameter 0) (color 0 0 0 0)
+  )
+  (junction (at 127 91.44) (diameter 0) (color 0 0 0 0)
+  )
+  (junction (at 128.27 127) (diameter 0) (color 0 0 0 0)
+  )
+  (junction (at 210.82 38.1) (diameter 0) (color 0 0 0 0)
+  )
+  (junction (at 92.71 157.48) (diameter 0) (color 0 0 0 0)
+  )
+  (junction (at 60.96 162.56) (diameter 0) (color 0 0 0 0)
+  )
+  (junction (at 118.11 137.16) (diameter 0) (color 0 0 0 0)
+  )
+  (junction (at 165.1 91.44) (diameter 0) (color 0 0 0 0)
+  )
+  (junction (at 165.1 86.36) (diameter 0) (color 0 0 0 0)
+  )
+  (junction (at 111.76 91.44) (diameter 0) (color 0 0 0 0)
+  )
+  (junction (at 92.71 139.7) (diameter 0) (color 0 0 0 0)
+  )
+  (junction (at 121.92 81.28) (diameter 0) (color 0 0 0 0)
+  )
+  (junction (at 105.41 30.48) (diameter 0) (color 0 0 0 0)
+  )
+  (junction (at 81.28 38.1) (diameter 0) (color 0 0 0 0)
+  )
+  (junction (at 71.12 134.62) (diameter 0) (color 0 0 0 0)
+  )
+  (junction (at 54.61 30.48) (diameter 0) (color 0 0 0 0)
+  )
+  (junction (at 106.68 81.28) (diameter 0) (color 0 0 0 0)
+  )
+  (junction (at 81.28 30.48) (diameter 0) (color 0 0 0 0)
+  )
+  (junction (at 55.88 91.44) (diameter 0) (color 0 0 0 0)
+  )
+  (junction (at 127 81.28) (diameter 0) (color 0 0 0 0)
+  )
+  (junction (at 129.54 41.91) (diameter 0) (color 0 0 0 0)
+  )
+  (junction (at 116.84 91.44) (diameter 0) (color 0 0 0 0)
+  )
+  (junction (at 171.45 130.81) (diameter 0) (color 0 0 0 0)
+  )
+  (junction (at 92.71 151.13) (diameter 0) (color 0 0 0 0)
   )
   (junction (at 87.63 81.28) (diameter 0) (color 0 0 0 0)
-  )
-  (junction (at 116.84 81.28) (diameter 0) (color 0 0 0 0)
-  )
-  (junction (at 128.27 132.08) (diameter 0) (color 0 0 0 0)
-  )
-  (junction (at 118.11 160.02) (diameter 0) (color 0 0 0 0)
-  )
-  (junction (at 60.96 134.62) (diameter 0) (color 0 0 0 0)
-  )
-  (junction (at 71.12 162.56) (diameter 0) (color 0 0 0 0)
-  )
-  (junction (at 106.68 91.44) (diameter 0) (color 0 0 0 0)
-  )
-  (junction (at 134.62 158.75) (diameter 0) (color 0 0 0 0)
-  )
-  (junction (at 127 91.44) (diameter 0) (color 0 0 0 0)
-  )
-  (junction (at 128.27 127) (diameter 0) (color 0 0 0 0)
-  )
-  (junction (at 161.29 130.81) (diameter 0) (color 0 0 0 0)
-  )
-  (junction (at 210.82 38.1) (diameter 0) (color 0 0 0 0)
-  )
-  (junction (at 92.71 157.48) (diameter 0) (color 0 0 0 0)
-  )
-  (junction (at 60.96 162.56) (diameter 0) (color 0 0 0 0)
-  )
-  (junction (at 118.11 137.16) (diameter 0) (color 0 0 0 0)
-  )
-  (junction (at 165.1 91.44) (diameter 0) (color 0 0 0 0)
-  )
-  (junction (at 165.1 86.36) (diameter 0) (color 0 0 0 0)
-  )
-  (junction (at 111.76 91.44) (diameter 0) (color 0 0 0 0)
-  )
-  (junction (at 92.71 139.7) (diameter 0) (color 0 0 0 0)
-  )
-  (junction (at 55.88 81.28) (diameter 0) (color 0 0 0 0)
-  )
-  (junction (at 161.29 146.05) (diameter 0) (color 0 0 0 0)
-  )
-  (junction (at 121.92 81.28) (diameter 0) (color 0 0 0 0)
-  )
-  (junction (at 105.41 30.48) (diameter 0) (color 0 0 0 0)
-  )
-  (junction (at 81.28 38.1) (diameter 0) (color 0 0 0 0)
-  )
-  (junction (at 71.12 134.62) (diameter 0) (color 0 0 0 0)
-  )
-  (junction (at 54.61 30.48) (diameter 0) (color 0 0 0 0)
-  )
-  (junction (at 106.68 81.28) (diameter 0) (color 0 0 0 0)
-  )
-  (junction (at 81.28 30.48) (diameter 0) (color 0 0 0 0)
-  )
-  (junction (at 55.88 91.44) (diameter 0) (color 0 0 0 0)
-  )
-  (junction (at 127 81.28) (diameter 0) (color 0 0 0 0)
-  )
-  (junction (at 129.54 41.91) (diameter 0) (color 0 0 0 0)
-  )
-  (junction (at 116.84 91.44) (diameter 0) (color 0 0 0 0)
-  )
-  (junction (at 171.45 130.81) (diameter 0) (color 0 0 0 0)
-  )
-  (junction (at 92.71 151.13) (diameter 0) (color 0 0 0 0)
   )
   (junction (at 105.41 41.91) (diameter 0) (color 0 0 0 0)
@@
     (stroke (width 0) (type default))
   )
-  (wire (pts (xy 62.23 106.68) (xy 92.71 106.68))
-    (stroke (width 0) (type default))
-  )
   (wire (pts (xy 71.12 133.35) (xy 71.12 134.62))
     (stroke (width 0) (type default))
@@
     (stroke (width 0) (type default))
   )
-  (wire (pts (xy 62.23 81.28) (xy 62.23 106.68))
-    (stroke (width 0) (type default))
-  )
   (wire (pts (xy 58.42 134.62) (xy 60.96 134.62))
     (stroke (width 0) (type default))
@@
     (stroke (width 0) (type default))
   )
+  (wire (pts (xy 63.5 83.82) (xy 63.5 106.68))
+    (stroke (width 0) (type default))
+  )
   (wire (pts (xy 87.63 90.17) (xy 87.63 91.44))
     (stroke (width 0) (type default))
@@
     (stroke (width 0) (type default))
   )
-  (wire (pts (xy 62.23 81.28) (xy 87.63 81.28))
-    (stroke (width 0) (type default))
-  )
   (wire (pts (xy 87.63 81.28) (xy 87.63 82.55))
     (stroke (width 0) (type default))
   )
-  (wire (pts (xy 55.88 81.28) (xy 62.23 81.28))
-    (stroke (width 0) (type default))
-  )
   (wire (pts (xy 116.84 160.02) (xy 118.11 160.02))
     (stroke (width 0) (type default))
@@
     (stroke (width 0) (type default))
   )
+  (wire (pts (xy 66.04 81.28) (xy 87.63 81.28))
+    (stroke (width 0) (type default))
+  )
   (wire (pts (xy 121.92 81.28) (xy 121.92 82.55))
     (stroke (width 0) (type default))
@@
     (stroke (width 0) (type default))
   )
+  (wire (pts (xy 63.5 106.68) (xy 92.71 106.68))
+    (stroke (width 0) (type default))
+  )
   (wire (pts (xy 120.65 152.4) (xy 120.65 157.48))
     (stroke (width 0) (type default))
@@
   )
   (wire (pts (xy 106.68 81.28) (xy 111.76 81.28))
+    (stroke (width 0) (type default))
+  )
+  (wire (pts (xy 55.88 81.28) (xy 60.96 81.28))
     (stroke (width 0) (type default))
   )
@@
     (pin "1")
   )
+  (symbol (lib_id "Device:NetTie_3_Tee") (at 63.5 81.28 0) (unit 1)
+    (in_bom yes) (on_board yes)
+    (default_instance (reference "NT") (unit 1) (value "NetTie_3_Tee") (footprint ""))
+    (property "Reference" "NT" (id 0) (at 66.04 82.55 0)
+      (effects (font (size 1.27 1.27)) hide)
+    )
+    (property "Value" "NetTie_3_Tee" (id 1) (at 63.5 80.0831 0)
+      (effects (font (size 1.27 1.27)) hide)
+    )
+    (property "Footprint" "" (id 2) (at 63.5 81.28 0)
+      (effects (font (size 1.27 1.27)) hide)
+    )
+    (property "Datasheet" "~" (id 3) (at 63.5 81.28 0)
+      (effects (font (size 1.27 1.27)) hide)
+    )
+    (pin "1")
+    (pin "2")
+    (pin "3")
+  )
   (symbol (lib_id "Connector:Conn_01x02_Female") (at 38.1 83.82 180) (unit 1)
     (in_bom yes) (on_board yes)
@@
     )
     (path "/65f64145-d9bc-4700-a819-90d988275300"
-      (reference "D2") (unit 1) (value "LED") (footprint "")
+      (reference "D2") (unit 1) (value "LED") (footprint "LED_SMD:LED_0805_2012Metric_Pad1.15x1.40mm_HandSolder")
     )
     (path "/7370e5a6-490f-4dfe-962a-df286192acc7"
@@
     )
     (path "/9419a865-ba34-432a-aebf-a54db959b750"
-      (reference "NT1") (unit 1) (value "NetTie_3_Tee") (footprint "NetTie:NetTie-3_THT_Pad1.0mm")
+      (reference "NT1") (unit 1) (value "NetTie_3_Tee") (footprint "NetTie:NetTie-3_SMD_Pad0.5mm")
     )
     (path "/18bbe3fa-16d5-41cc-a681-f01d6e2b1783"
-      (reference "NT2") (unit 1) (value "NetTie_3_Tee") (footprint "NetTie:NetTie-3_THT_Pad1.0mm")
+      (reference "NT2") (unit 1) (value "NetTie_3_Tee") (footprint "NetTie:NetTie-3_SMD_Pad0.5mm")
+    )
+    (path "/72c850f3-4227-4466-bc48-042adc122ab1"
+      (reference "NT?") (unit 1) (value "NetTie_3_Tee") (footprint "NetTie:NetTie-3_SMD_Pad0.5mm")
     )
     (path "/2cbae96b-ac89-47c9-b39b-124ad157f172"
@@
     )
     (path "/f132667e-014d-4086-bf0b-1ab1d8c8cb39"
-      (reference "TP1") (unit 1) (value "Sweep Hi PWM") (footprint "")
+      (reference "TP1") (unit 1) (value "Sweep Hi PWM") (footprint "TestPoint:TestPoint_Pad_D2.0mm")
     )
     (path "/c7296472-cdb9-4ce0-ae36-e88c86934623"
-      (reference "TP2") (unit 1) (value "Sweep Lo PWM") (footprint "")
+      (reference "TP2") (unit 1) (value "Sweep Lo PWM") (footprint "TestPoint:TestPoint_Pad_D2.0mm")
     )
     (path "/4caa870c-42bb-495f-ba41-df04e97b661b"
-      (reference "TP3") (unit 1) (value "Sweep Hi Analog") (footprint "")
+      (reference "TP3") (unit 1) (value "Sweep Hi Analog") (footprint "TestPoint:TestPoint_Pad_D2.0mm")
     )
     (path "/ca096f3d-c400-4f7c-9d6f-d80e4f498d19"
-      (reference "TP4") (unit 1) (value "Sweep Lo Analog") (footprint "")
+      (reference "TP4") (unit 1) (value "Sweep Lo Analog") (footprint "TestPoint:TestPoint_Pad_D2.0mm")
     )
     (path "/0aeeae37-f5df-48bf-84c7-1d9ba9d4c49f"
-      (reference "TP5") (unit 1) (value "Voltage Sense Div") (footprint "")
+      (reference "TP5") (unit 1) (value "Voltage Sense Div") (footprint "TestPoint:TestPoint_Pad_D2.0mm")
     )
     (path "/0744d3b7-ccbd-4377-83e4-b9b58a44add3"
-      (reference "TP6") (unit 1) (value "Gate Drv Out") (footprint "")
+      (reference "TP6") (unit 1) (value "Gate Drv Out") (footprint "TestPoint:TestPoint_Pad_D2.0mm")
     )
     (path "/c797a0e8-4edf-450c-b463-6868853c02cf"
-      (reference "TP7") (unit 1) (value "Gate Drv In") (footprint "")
+      (reference "TP7") (unit 1) (value "Gate Drv In") (footprint "TestPoint:TestPoint_Pad_D2.0mm")
     )
     (path "/78c5758c-1346-45ea-808e-3af62c0f0e48"
