File: board/optimizer.kicad_sch (KiCad schematic)
At the start: 63 parts

Commit message: WIP
Parts:
- removed C (x6): C, symbol Device:C
- removed C (x7): C_Polarized, symbol Device:C_Polarized
- removed J (x2): Conn_01x02_Female, symbol Connector:Conn_01x02_Female
- removed NT (x3): NetTie_3_Tee, symbol Device:NetTie_3_Tee
- removed R (x10): R, symbol Device:R
- removed TP (x5): TestPoint_Probe, symbol Connector:TestPoint_Probe
- removed U (x5): 74HC00, symbol 74xx:74HC00
- removed U (x3): LM393, symbol Comparator:LM393
- removed U: ATSAMD10D14A-SS, Package_SO:SOIC-20W_7.5x12.8mm_P1.27mm, symbol MCU_Microchip_SAMD:ATSAMD10D14A-SS
- removed U: LM1117-3.3, symbol Regulator_Linear:LM1117-3.3
- added C (x21): C, symbol Device:C_Small
- added C (x4): C, symbol Device:C
- added D (x2): BAT54S, Package_TO_SOT_SMD:SOT-23, symbol Diode:BAT54S
- added J (x4): Conn_01x01_Female, symbol Connector:Conn_01x01_Female
- added L: L, symbol Device:L
- added NT (x4): NetTie_2, symbol Device:NetTie_2
- added R (x5): R, symbol Device:R
- added TP (x3): TestPoint_Probe, symbol Connector:TestPoint_Probe
- added U: ATSAMD09C13A-SS, Package_SO:SOIC-14_3.9x8.7mm_P1.27mm, symbol MCU_Microchip_SAMD:ATSAMD09C13A-SS
- added U: RT9193, symbol Drake:RT9193
- L: TME DTMSS-20/0.010/20-V -> https://www.tme.eu/cz/details/de1207-1/vykonne-tlumivky-smd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
Connections:
- net +12V: now also U.1 (VIN)
- net +3V3: now also C.1, D.2, D.2, U.12 (VDD), U.5 (VOUT)
- net GND: now also C.2, C.2, C.2, C.2, D.1, D.1, NT.1, R.2, R.2, U.11 (GND), U.2 (GND), U.3 (EN); no longer C.2, C.2, C.2, C.2, R.2, U.4 (GND)
- net LED: now also U.2 (PA08/XIN)
- net SWITCH_PATH2: now reaches Q.1 (G), TP.1, U.5 (OUT)
- net PWR_IN: now reaches L.1
- net PWR_IN: now also C.2, C.2, C.2, C.2, C.2, C.2, C.2, C.2, C.2, C.2, J.1 (Pin_1), NT.1, NT.1; no longer D.1 (K)
- net PWR_PATH1: now reaches L.2
- net PWR_PATH1: now also Q.2 (D), C.1
- net SWITCH_PATH1: now reaches C.1, U.3 (VI)
- net SWITCH_PATH1: now also NT.2
- net PWR_GND: now reaches Q.3 (S)
- net PWR_GND: now also C.2, C.2, C.2, C.2, R.2, U.4 (GND), C.1, C.1, C.1, C.1, C.1, C.1, C.1, C.1, C.1, C.1, C.1, C.1, C.1, C.1, C.1, C.1, C.1, C.1, C.1, C.1, J.1 (Pin_1), J.1 (Pin_1), L.2, NT.2; no longer D.2 (A)
- net at C.2: now also U.6 (PA28/~{RST})
- net at X.3 (SWCLK): now also U.7 (PA30/SWCLK)
- net at X.1 (SWDIO): now also U.8 (PA31/SWDIO)
- net GATE: now reaches U.3 (IN)
- net GATE: now also TP.1, U.9 (PA24)
- net TEL1 renamed TELEMETRY_1
- net TELEMETRY_1: now also U.4 (PA14)
- net TEL2 renamed TELEMETRY_2
- net TELEMETRY_2: now also U.5 (PA15)
- new net: C.1, U.4 (BP)
- new net: R.1, R.2
- new net PWR_OUT: C.2, C.2, C.2, C.2, C.2, C.2, C.2, C.2, C.2, C.2, D.1 (K), J.1 (Pin_1), NT.1
- new net PWR_PATH2: C.2, D.2 (A), L.1
- new net V_IN_FULL: NT.2, R.1
- new net V_IN_SCALE: C.1, D.3, R.1, R.2, TP.1, U.13 (PA02)
- new net V_OUT_FULL: NT.2, R.1
- new net V_OUT_SCALE: C.1, D.3, R.1, R.2, TP.1, U.14 (PA04)
- no-connect marks 5 -> 3
Other:
- moved on the sheet: C, D, J, L, Q, TP, U

Commit message: WIP
Connections:
- net +12V: now also U.3 (EN)
- net GATE: now also U.1 (PA05); no longer U.9 (PA24)
- net GND: no longer U.3 (EN)
Changed lines of the file:
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@@
   (junction (at 93.345 166.37) (diameter 0) (color 0 0 0 0)
+  )
+  (junction (at 110.49 41.91) (diameter 0) (color 0 0 0 0)
   )
   (junction (at 64.77 91.44) (diameter 0) (color 0 0 0 0)
@@
   (no_connect (at 229.87 66.04))
   (no_connect (at 255.27 66.04))
-  (no_connect (at 255.27 55.88))
+  (no_connect (at 255.27 63.5))
   (wire (pts (xy 212.09 59.69) (xy 222.25 59.69))
     (stroke (width 0) (type default))
@@
     (stroke (width 0) (type default))
   )
+  (wire (pts (xy 110.49 41.91) (xy 110.49 49.53))
+    (stroke (width 0) (type default))
+  )
   (wire (pts (xy 76.2 132.08) (xy 80.01 132.08))
     (stroke (width 0) (type default))
@@
   )
   (wire (pts (xy 57.15 132.08) (xy 60.96 132.08))
-    (stroke (width 0) (type default))
-  )
-  (wire (pts (xy 110.49 57.15) (xy 110.49 49.53))
     (stroke (width 0) (type default))
   )
@@
     (effects (font (size 1.27 1.27)) (justify left bottom))
   )
-  (label "GATE" (at 255.27 63.5 0) (fields_autoplaced)
+  (label "GATE" (at 255.27 55.88 0) (fields_autoplaced)
     (effects (font (size 1.27 1.27)) (justify left bottom))
   )
@@
   )
   (symbol (lib_id "Device:C") (at 105.41 45.72 0) (unit 1)
-    (in_bom yes) (on_board yes) (fields_autoplaced)
-    (default_instance (reference "C") (unit 1) (value "C") (footprint ""))
-    (property "Reference" "C" (id 0) (at 108.331 45.1255 0)
-      (effects (font (size 1.27 1.27)) (justify left))
-    )
-    (property "Value" "C" (id 1) (at 108.331 46.8877 0)
+    (in_bom yes) (on_board yes)
+    (default_instance (reference "C") (unit 1) (value "C") (footprint ""))
+    (property "Reference" "C" (id 0) (at 99.06 44.45 0)
+      (effects (font (size 1.27 1.27)) (justify left))
+    )
+    (property "Value" "C" (id 1) (at 99.06 46.355 0)
       (effects (font (size 1.27 1.27)) (justify left))
     )
@@
     )
     (property "Datasheet" "~" (id 3) (at 31.75 33.02 0)
-      (effects (font (size 1.27 1.27)) hide)
-    )
-    (pin "1")
-  )
-  (symbol (lib_id "power:GND") (at 110.49 57.15 0) (unit 1)
-    (in_bom yes) (on_board yes) (fields_autoplaced)
-    (default_instance (reference "#PWR") (unit 1) (value "GND") (footprint ""))
-    (property "Reference" "#PWR" (id 0) (at 110.49 63.5 0)
-      (effects (font (size 1.27 1.27)) hide)
-    )
-    (property "Value" "GND" (id 1) (at 110.49 61.2061 0)
-      (effects (font (size 1.27 1.27)))
-    )
-    (property "Footprint" "" (id 2) (at 110.49 57.15 0)
-      (effects (font (size 1.27 1.27)) hide)
-    )
-    (property "Datasheet" "" (id 3) (at 110.49 57.15 0)
       (effects (font (size 1.27 1.27)) hide)
     )
@@
       (reference "#PWR013") (unit 1) (value "+12V") (footprint "")
     )
-    (path "/fadabf4b-c917-424b-a1cb-2199970a8a8d"
-      (reference "#PWR014") (unit 1) (value "GND") (footprint "")
-    )
     (path "/511cbf92-4000-415d-8912-e3f2dbd1d1b8"
       (reference "#PWR015") (unit 1) (value "GND") (footprint "")
@@
     )
     (path "/48c18c2b-6d18-4754-a76e-01daceb57b76"
-      (reference "U3") (unit 1) (value "RT9193") (footprint "Package_TO_SOT_SMD:SOT-23-5_HandSoldering")
+      (reference "U3") (unit 1) (value "SPX3819") (footprint "Package_TO_SOT_SMD:SOT-23-5_HandSoldering")
     )
     (path "/4289a6dd-e222-4311-8514-5facfc0b2875"

Commit message: WIP
Parts:
- removed C: C, symbol Device:C
- removed R: R, symbol Device:R
- removed U: RT9193, symbol Drake:RT9193
- added U: AP1117-33, Package_TO_SOT_SMD:SOT-223-3_TabPin2, symbol Regulator_Linear:AP1117-33
Connections:
- net +12V: now also U.3 (VI)
- net +3V3: now also U.2 (VO)
- net GND: now also U.1 (GND)
- net V_OUT_SCALE: now also R.2
Other:
- moved on the sheet: R

Commit message: WIP
Changed lines of the file:
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@@
-    (pin "1")
-  )
-  (symbol (lib_id "power:+3V3") (at 31.75 33.02 270) (unit 1)
-    (in_bom yes) (on_board yes) (fields_autoplaced)
-    (default_instance (reference "#PWR") (unit 1) (value "+3V3") (footprint ""))
-    (property "Reference" "#PWR" (id 0) (at 27.94 33.02 0)
-      (effects (font (size 1.27 1.27)) hide)
-    )
-    (property "Value" "+3V3" (id 1) (at 34.925 33.3066 90)
-      (effects (font (size 1.27 1.27)) (justify left))
-    )
-    (property "Footprint" "" (id 2) (at 31.75 33.02 0)
-      (effects (font (size 1.27 1.27)) hide)
-    )
-    (property "Datasheet" "" (id 3) (at 31.75 33.02 0)
-      (effects (font (size 1.27 1.27)) hide)
-    )
     (pin "1")
   )
@@
     (pin "1")
   )
-  (symbol (lib_id "power:PWR_FLAG") (at 31.75 33.02 90) (unit 1)
-    (in_bom yes) (on_board yes) (fields_autoplaced)
-    (default_instance (reference "#FLG") (unit 1) (value "PWR_FLAG") (footprint ""))
-    (property "Reference" "#FLG" (id 0) (at 29.845 33.02 0)
-      (effects (font (size 1.27 1.27)) hide)
-    )
-    (property "Value" "PWR_FLAG" (id 1) (at 28.5751 33.3066 90)
-      (effects (font (size 1.27 1.27)) (justify left))
-    )
-    (property "Footprint" "" (id 2) (at 31.75 33.02 0)
-      (effects (font (size 1.27 1.27)) hide)
-    )
-    (property "Datasheet" "~" (id 3) (at 31.75 33.02 0)
-      (effects (font (size 1.27 1.27)) hide)
-    )
-    (pin "1")
-  )
   (sheet_instances
     (path "/" (page "1"))
   )
   (symbol_instances
-    (path "/f7d214c0-3112-4323-976f-def2e85c4b69"
-      (reference "#FLG01") (unit 1) (value "PWR_FLAG") (footprint "")
-    )
     (path "/3889ce09-ac85-490f-87ba-3af56aea98a6"
       (reference "#FLG02") (unit 1) (value "PWR_FLAG") (footprint "")
@@
       (reference "#FLG0101") (unit 1) (value "PWR_FLAG") (footprint "")
     )
-    (path "/c0a47382-b6e3-4ddf-99b2-bf7c716b2a39"
-      (reference "#PWR01") (unit 1) (value "+3V3") (footprint "")
-    )
     (path "/e7b94e1f-1f0b-402e-988e-668013710a5c"
       (reference "#PWR02") (unit 1) (value "GND") (footprint "")
@@
       (reference "U2") (unit 1) (value "LM317_TO-252") (footprint "Package_TO_SOT_SMD:TO-252-2")
     )
+    (path "/348df945-ad6d-4d47-b930-3dfbe85d5468"
+      (reference "U3") (unit 1) (value "AP1117-33") (footprint "Package_TO_SOT_SMD:SOT-223-3_TabPin2")
+    )
     (path "/4289a6dd-e222-4311-8514-5facfc0b2875"
       (reference "U4") (unit 1) (value "ATSAMD09C13A-SS") (footprint "Package_SO:SOIC-14_3.9x8.7mm_P1.27mm")
     )
-    (path "/348df945-ad6d-4d47-b930-3dfbe85d5468"
-      (reference "U?") (unit 1) (value "AP1117-33") (footprint "Package_TO_SOT_SMD:SOT-223-3_TabPin2")
-    )
     (path "/be4ac40d-90a1-4523-85d9-2abd4bd40819"

Commit message: WIP
Parts:
- removed C (x16): C, symbol Device:C_Small
- removed C: C, symbol Device:C
- removed D: BAT54S, Package_TO_SOT_SMD:SOT-23, symbol Diode:BAT54S
- removed L (x2): L, symbol Device:L
- removed NT: NetTie_2, symbol Device:NetTie_2
- removed R (x2): R, symbol Device:R
- removed TP: TestPoint_Probe, symbol Connector:TestPoint_Probe
- removed U: MCP1416, Package_TO_SOT_SMD:SOT-23-5, symbol Driver_FET:MCP1416
- added C: C, symbol Device:C_Small
- added H (x2): MountingHole, symbol Mechanical:MountingHole
- added U: ZXGD3009E6, Package_TO_SOT_SMD:SOT-23-6, symbol Driver_FET:ZXGD3009E6
Connections:
- net PWR_OUT is gone; now on net PWR_P: C.2, C.2, C.2, C.2, C.2, D.1 (K), J.1 (Pin_1)
- net PWR_PATH2 is gone; now on net PWR_GND_OUT: D.2 (A)
- net +12V: now also U.1 (VCC)
- net PWR_GND: now also C.1, U.3 (VEE); no longer J.1 (Pin_1)
- net GATE renamed GATE_LOG
- net GATE_LOG: now also U.2 (IN)
- net PWR_IN renamed PWR_P
- net PWR_P: now also C.2
- net PWR_PATH1 renamed PWR_GND_OUT
- net PWR_GND_OUT: now also J.1 (Pin_1)
- net SWITCH_PATH2 renamed GATE_PWR
- net GATE_PWR: now also U.4 (SINK), U.6 (SOURCE)
- net V_IN_FULL renamed V_FULL
- net V_IN_SCALE renamed V_SCALE
- net V_OUT_SCALE: no longer names the net of U.14 (PA04)
- no-connect marks 3 -> 4
Other:
- moved on the sheet: C, D, J, NT, Q, R, TP
