File: board/optimizer.kicad_pcb (KiCad board)
At the start: 0 parts

Commit message: WIP
Parts:
- added C1: 100n, Capacitor_SMD:C_0805_2012Metric_Pad1.18x1.45mm_HandSolder, F.Cu at (115.0, 131.0)
- added C10: 10u/50V, Capacitor_SMD:C_1206_3216Metric_Pad1.33x1.80mm_HandSolder, F.Cu at (126.5, 140.0)
- added C11: 10u/50V, Capacitor_SMD:C_1206_3216Metric_Pad1.33x1.80mm_HandSolder, F.Cu at (123.5, 140.0)
- added C12: 100n, Capacitor_SMD:C_0805_2012Metric_Pad1.18x1.45mm_HandSolder, F.Cu at (181.0, 132.0)
- added C13: 1u, Capacitor_SMD:C_0805_2012Metric_Pad1.18x1.45mm_HandSolder, F.Cu at (181.0, 134.5)
- added C14: 1u, Capacitor_SMD:C_0805_2012Metric_Pad1.18x1.45mm_HandSolder, F.Cu at (115.0, 126.0)
- added C15: 1u, Capacitor_SMD:C_0805_2012Metric_Pad1.18x1.45mm_HandSolder, F.Cu at (126.5, 134.0)
- added C16: 10u/50V, Capacitor_SMD:C_1206_3216Metric_Pad1.33x1.80mm_HandSolder, F.Cu at (160.0, 120.0)
- added C17: 10u/50V, Capacitor_SMD:C_1206_3216Metric_Pad1.33x1.80mm_HandSolder, F.Cu at (168.5, 95.4)
- added C18: 10u/50V, Capacitor_SMD:C_1206_3216Metric_Pad1.33x1.80mm_HandSolder, F.Cu at (171.5, 95.4)
- added C19: 10u/50V, Capacitor_SMD:C_1206_3216Metric_Pad1.33x1.80mm_HandSolder, F.Cu at (174.5, 95.4)
- added C2: 10u/50V, Capacitor_SMD:C_1206_3216Metric_Pad1.33x1.80mm_HandSolder, F.Cu at (150.5, 140.0)
- added C20: 10u/50V, Capacitor_SMD:C_1206_3216Metric_Pad1.33x1.80mm_HandSolder, F.Cu at (177.5, 95.4)
- added C21: 10u/50V, Capacitor_SMD:C_1206_3216Metric_Pad1.33x1.80mm_HandSolder, F.Cu at (180.5, 95.4)
- added C22: 10u/50V, Capacitor_SMD:C_1206_3216Metric_Pad1.33x1.80mm_HandSolder, F.Cu at (183.5, 95.4)
- added C23: 10u/50V, Capacitor_SMD:C_1206_3216Metric_Pad1.33x1.80mm_HandSolder, F.Cu at (186.5, 95.4)
- added C24: 10u/50V, Capacitor_SMD:C_1206_3216Metric_Pad1.33x1.80mm_HandSolder, F.Cu at (189.5, 95.4)
- added C25: 10u/50V, Capacitor_SMD:C_1206_3216Metric_Pad1.33x1.80mm_HandSolder, F.Cu at (192.5, 95.4)
- added C26: 10u/50V, Capacitor_SMD:C_1206_3216Metric_Pad1.33x1.80mm_HandSolder, F.Cu at (195.5, 95.4)
- added C27: 22n, Capacitor_SMD:C_0805_2012Metric_Pad1.18x1.45mm_HandSolder, F.Cu at (117.0, 135.5)
- added C28: 1u, Capacitor_SMD:C_0805_2012Metric_Pad1.18x1.45mm_HandSolder, F.Cu at (119.5, 138.5)
- added C29: 100n, Capacitor_SMD:C_0805_2012Metric_Pad1.18x1.45mm_HandSolder, F.Cu at (199.5, 129.0)
- added C3: 10u/50V, Capacitor_SMD:C_1206_3216Metric_Pad1.33x1.80mm_HandSolder, F.Cu at (147.5, 140.0)
- added C30: 100n, Capacitor_SMD:C_0805_2012Metric_Pad1.18x1.45mm_HandSolder, F.Cu at (188.5, 134.0)
- added C31: 1u, Capacitor_SMD:C_0805_2012Metric_Pad1.18x1.45mm_HandSolder, F.Cu at (186.0, 134.0)
- added C32: 100n, Capacitor_SMD:C_0805_2012Metric_Pad1.18x1.45mm_HandSolder, F.Cu at (199.5, 135.5)
- added C33: 100n, Capacitor_SMD:C_0805_2012Metric_Pad1.18x1.45mm_HandSolder, F.Cu at (220.2, 112.2)
- added C4: 10u/50V, Capacitor_SMD:C_1206_3216Metric_Pad1.33x1.80mm_HandSolder, F.Cu at (144.5, 140.0)
- added C5: 10u/50V, Capacitor_SMD:C_1206_3216Metric_Pad1.33x1.80mm_HandSolder, F.Cu at (141.5, 140.0)
- added C6: 10u/50V, Capacitor_SMD:C_1206_3216Metric_Pad1.33x1.80mm_HandSolder, F.Cu at (138.5, 140.0)
- added C7: 10u/50V, Capacitor_SMD:C_1206_3216Metric_Pad1.33x1.80mm_HandSolder, F.Cu at (135.5, 140.0)
- added C8: 10u/50V, Capacitor_SMD:C_1206_3216Metric_Pad1.33x1.80mm_HandSolder, F.Cu at (132.5, 140.0)
- added C9: 10u/50V, Capacitor_SMD:C_1206_3216Metric_Pad1.33x1.80mm_HandSolder, F.Cu at (129.5, 140.0)
- added D1: DSS16-01AS, Package_TO_SOT_SMD:TO-263-2_TabPin1, F.Cu at (169.6, 111.0)
- added D2: LED, LED_SMD:LED_0805_2012Metric_Pad1.15x1.40mm_HandSolder, F.Cu at (217.0, 121.0)
- added D3: BAT54S, Package_TO_SOT_SMD:SOT-23, F.Cu at (220.0, 136.5)
- added D4: BAT54S, Package_TO_SOT_SMD:SOT-23, F.Cu at (220.3, 108.5)
- added J1: Telemetry, Connector_PinHeader_2.54mm:PinHeader_1x04_P2.54mm_Vertical, F.Cu at (203.0, 136.3)
- added J2: IN+, optimizer:Wire 4mm2, F.Cu at (140.0, 130.5)
- added J3: IN-, optimizer:Wire 4mm2, F.Cu at (173.0, 140.0)
- added J4: OUT-, optimizer:Wire 4mm2, F.Cu at (156.0, 101.0)
- added J5: OUT+, optimizer:Wire 4mm2, F.Cu at (164.0, 101.0)
- added L1: 1uH/14A, Inductor_SMD:L_12x12mm_H8mm, F.Cu at (151.0, 129.0)
- added L2: 1uH/14A, Inductor_SMD:L_12x12mm_H8mm, F.Cu at (169.0, 129.0)
- added NT1: NetTie_2, optimizer:NetTie 1 mm, F.Cu at (135.8, 126.8)
- added NT2: NetTie_2, optimizer:NetTie 0.4 mm, F.Cu at (115.2, 132.5)
- added NT3: NetTie_2, optimizer:NetTie 0.4 mm, F.Cu at (135.0, 135.2)
- added NT4: NetTie_2, optimizer:NetTie 0.4 mm, F.Cu at (224.1, 110.0)
- added Q1: AOB2500L, Package_TO_SOT_SMD:TO-263-2, F.Cu at (150.4, 111.0)
- added R1: 4k5, Resistor_SMD:R_0805_2012Metric_Pad1.20x1.40mm_HandSolder, F.Cu at (189.5, 139.0)
- added R2: 270R, Resistor_SMD:R_0805_2012Metric_Pad1.20x1.40mm_HandSolder, F.Cu at (119.0, 128.5)
- added R3: 2k26, Resistor_SMD:R_0805_2012Metric_Pad1.20x1.40mm_HandSolder, F.Cu at (115.0, 128.5)
- added R4: 270R, Resistor_SMD:R_0805_2012Metric_Pad1.20x1.40mm_HandSolder, F.Cu at (199.0, 139.0)
- added R5: 270R, Resistor_SMD:R_0805_2012Metric_Pad1.20x1.40mm_HandSolder, F.Cu at (217.0, 125.0)
- added R6: 4k5, Resistor_SMD:R_0805_2012Metric_Pad1.20x1.40mm_HandSolder, F.Cu at (229.9, 107.8)
- added R7: 4k5, Resistor_SMD:R_0805_2012Metric_Pad1.20x1.40mm_HandSolder, F.Cu at (225.1, 107.8)
- added R8: 270R, Resistor_SMD:R_0805_2012Metric_Pad1.20x1.40mm_HandSolder, F.Cu at (225.0, 112.2)
- added TP1: Gate Log, TestPoint:TestPoint_Pad_D2.0mm, F.Cu at (188.5, 125.0)
- added TP2: Voltage Sense, TestPoint:TestPoint_Pad_D2.0mm, F.Cu at (184.0, 138.0)
- added TP3: Gate Pwr, TestPoint:TestPoint_Pad_D2.0mm, F.Cu at (185.0, 125.0)
- added TP4: Voltage Sense, TestPoint:TestPoint_Pad_D2.0mm, F.Cu at (229.4, 111.3)
- added U1: MCP1416, Package_TO_SOT_SMD:SOT-23-5, F.Cu at (183.5, 128.0)
- added U2: LM317_TO-252, Package_TO_SOT_SMD:TO-252-2, F.Cu at (130.1, 129.0)
- added U3: RT9193, Package_TO_SOT_SMD:SOT-23-5_HandSoldering, F.Cu at (120.0, 134.5)
- added U4: ATSAMD09C13A-SS, Package_SO:SOIC-14_3.9x8.7mm_P1.27mm, F.Cu at (194.0, 133.0)
- added X1: SWD, Drake:SWD, F.Cu at (194.0, 126.5)
Routing:
- net +12V: track 0.00 -> 115.9 mm, vias 0 -> 2
- net /V_IN_FULL: track 0.00 -> 59.6 mm, vias 0 -> 2
- net GND: track 0.00 -> 55.5 mm, vias 0 -> 2
- net /SWITCH_PATH2: track 0.00 -> 47.7 mm, vias 0 -> 3
- net Net-(U2-ADJ): track 0.00 -> 24.2 mm, vias 0 -> 2
- net /SWITCH_PATH1: track 0.00 -> 20.3 mm, vias 0 -> 2
- net /V_IN_SCALE: track 0.00 -> 13.7 mm
- net /GATE: track 0.00 -> 11.2 mm
- net +3V3: track 0.00 -> 8.66 mm
- net /TELEMETRY_1: track 0.00 -> 6.84 mm
- net /TELEMETRY_2: track 0.00 -> 6.74 mm
- net Net-(U4-PA28/~{RST}): track 0.00 -> 3.20 mm
- net Net-(U4-PA31/SWDIO): track 0.00 -> 2.72 mm
- net Net-(U4-PA30/SWCLK): track 0.00 -> 2.72 mm
- net Net-(U3-BP): track 0.00 -> 2.62 mm
- added copper zone on F.Cu, net /PWR_GND
- added copper zone on F.Cu, net /PWR_IN
- added copper zone on F.Cu, net /PWR_OUT
- added copper zone on F.Cu, net /PWR_PATH1
- added copper zone on F.Cu, net /PWR_PATH2
Other:
- board outline added: 100 x 55 mm
- copper layers 0 -> 2

Commit message: WIP
Parts:
- moved C26 86.4 mm to (113.0, 121.0), turned to 90 degrees
- moved C25 80.7 mm to (116.0, 121.0), turned to 90 degrees
- moved C24 75.0 mm to (119.0, 121.0), turned to 90 degrees
- moved C23 69.4 mm to (122.0, 121.0), turned to 90 degrees
- moved NT4 65.6 mm to (158.5, 109.5)
- moved C22 63.8 mm to (125.0, 121.0), turned to 90 degrees
- moved C21 58.4 mm to (128.0, 121.0), turned to 90 degrees
- moved R6 57.9 mm to (178.0, 133.5)
- moved D3 56.5 mm to (163.5, 137.0)
- moved J2 55.4 mm to (194.5, 120.8)
- moved R7 54.6 mm to (179.0, 137.0), turned to -90 degrees
- moved R8 54.6 mm to (179.0, 141.5), turned to -90 degrees
- moved TP4 54.0 mm to (182.0, 137.0)
- moved D4 53.1 mm to (175.5, 137.0)
- moved C20 53.1 mm to (131.0, 121.0), turned to 90 degrees
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Routing:
- net +12V: track 115.9 -> 0.00 mm, vias 2 -> 0
- net /V_IN_FULL: track 59.6 -> 0.00 mm, vias 2 -> 0
- net GND: track 55.5 -> 0.00 mm, vias 2 -> 0
- net /SWITCH_PATH2: track 47.7 -> 0.00 mm, vias 3 -> 0
- net Net-(U2-ADJ): track 24.2 -> 0.00 mm, vias 2 -> 0
- net /SWITCH_PATH1: track 20.3 -> 0.00 mm, vias 2 -> 0
- net /V_IN_SCALE: track 13.7 -> 0.00 mm
- net /GATE: track 11.2 -> 0.00 mm
- net +3V3: track 8.66 -> 0.00 mm
- net /TELEMETRY_1: track 6.84 -> 0.00 mm
- net /TELEMETRY_2: track 6.74 -> 0.00 mm
- net Net-(U4-PA28/~{RST}): track 3.20 -> 0.00 mm
- net Net-(U4-PA31/SWDIO): track 2.72 -> 0.00 mm
- net Net-(U4-PA30/SWCLK): track 2.72 -> 0.00 mm
- net Net-(U3-BP): track 2.62 -> 0.00 mm
- added copper zone on F.Cu, net /SWITCH_PATH2

Commit message: WIP
Parts:
- moved R5 13.0 mm to (191.0, 142.5), turned to 180 degrees
- moved TP1 8.86 mm to (158.0, 140.0)
- moved C29 6.50 mm to (204.0, 141.5), turned to 90 degrees
- moved TP3 4.92 mm to (153.0, 135.5)
- moved U1 3.50 mm to (157.0, 135.0)
- moved C14 3.00 mm to (142.5, 132.5)
- moved R3 3.00 mm to (139.5, 132.5)
- moved NT1 2.50 mm to (161.0, 120.0)
- moved R2 1.58 mm to (141.0, 136.5), turned to 180 degrees
- moved C27 1.00 mm to (114.5, 134.0)
- moved D2 1.00 mm to (186.5, 142.5)
- moved C30 0.50 mm to (192.5, 139.0)
- turned X1 to 180 degrees
Routing:
- net +3V3: track 0.00 -> 58.2 mm
- net /SWITCH_PATH1: track 0.00 -> 54.7 mm, vias 0 -> 4
- net /SWITCH_PATH2: track 0.00 -> 49.7 mm, vias 0 -> 2
- net /V_OUT_FULL: track 0.00 -> 47.2 mm, vias 0 -> 2
- net /GATE: track 0.00 -> 43.2 mm, vias 0 -> 2
- net /V_IN_SCALE: track 0.00 -> 40.2 mm, vias 0 -> 2
- net GND: track 0.00 -> 35.6 mm, vias 0 -> 11
- net /V_OUT_SCALE: track 0.00 -> 27.7 mm, vias 0 -> 2
- net /V_IN_FULL: track 0.00 -> 22.2 mm, vias 0 -> 2
- net Net-(U4-PA30/SWCLK): track 0.00 -> 15.4 mm, vias 0 -> 1
- net Net-(U4-PA28/~{RST}): track 0.00 -> 11.9 mm, vias 0 -> 2
- net /LED: track 0.00 -> 11.0 mm
- net Net-(U2-ADJ): track 0.00 -> 10.4 mm
- net +12V: track 0.00 -> 9.16 mm
- net /TELEMETRY_1: track 0.00 -> 7.46 mm
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- added copper zone on F.Cu, net +12V
- added copper zone on F.Cu, net +3V3
- added copper zone on B.Cu, net /PWR_OUT
- added copper zone on B.Cu, net /PWR_PATH1
- added copper zone on B.Cu, net GND

Commit message: WIP
Parts:
- moved J2 1.50 mm to (196.0, 120.8)
- moved J3 1.50 mm to (196.0, 128.5)
- moved J5 1.00 mm to (125.0, 114.5)
- moved L1 0.50 mm to (170.0, 113.0)
Routing:
- net /V_OUT_FULL: track 47.2 -> 62.7 mm
- net /PWR_OUT: track 0.00 -> 4.84 mm, vias 0 -> 81
- net /SWITCH_PATH2: track 49.7 -> 52.0 mm
- net /PWR_IN: track 0.00 -> 2.21 mm
- net GND: track 35.6 -> 34.9 mm
- net /PWR_PATH1: vias 0 -> 76

Commit message: WIP
Parts:
- TP2: value Voltage Sense -> Volt. In Scaled
- TP4: value Voltage Sense -> Volt. Out Scaled
- moved TP4 1.00 mm to (182.0, 136.0)
Routing:
- net /V_OUT_SCALE: track 27.7 -> 28.7 mm
Other:
- board text added: "OPTIMIST v1.0"

Commit message: WIP
Parts:
- TP2: value Volt. In Scaled -> VIN Scaled
- TP4: value Volt. Out Scaled -> VOUT Scaled
- moved D1 1.00 mm to (135.0, 108.4)
- moved Q1 1.00 mm to (185.0, 108.4)
Routing:
- net /PWR_PATH1: vias 76 -> 78
- net /PWR_OUT: vias 81 -> 84
Changed lines of the file:
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@@
   )
   (footprint "Package_TO_SOT_SMD:TO-263-2_TabPin1" locked (layer "F.Cu")
-    (at 136 108.375 90)
+    (at 135 108.375 90)
     (descr "TO-263 / D2PAK / DDPAK SMD package, tab to pin 1, https://www.wolfspeed.com/media/downloads/137/C3D06060G.pdf")
     (tags "D2PAK DDPAK TO-263 D2PAK-3 TO-263-3 SOT-404 diode")
@@
         (effects (font (size 1 1) (thickness 0.15)))
     )
-    (fp_text value "Volt. Out Scaled" (at 4.25 -4.25 45) (layer "F.SilkS")
-        (effects (font (size 0.7 0.7) (thickness 0.1)))
+    (fp_text value "VOUT Scaled" (at 4.25 -4.25 45) (layer "F.SilkS")
+        (effects (font (size 1 1) (thickness 0.15)))
     )
     (fp_text user "${REFERENCE}" (at 0 -2) (layer "F.Fab")
@@
         (effects (font (size 1 1) (thickness 0.15)))
     )
-    (fp_text value "Gate Pwr" (at -3 3 45) (layer "F.SilkS")
-        (effects (font (size 0.7 0.7) (thickness 0.1)))
+    (fp_text value "Gate Pwr" (at -1.5 -1 45) (layer "F.SilkS")
+        (effects (font (size 1 1) (thickness 0.15)))
     )
     (fp_text user "${REFERENCE}" (at 0 -2) (layer "F.Fab")
@@
         (effects (font (size 1 1) (thickness 0.15)))
     )
-    (fp_text value "Volt. In Scaled" (at 3.75 -3.75 45) (layer "F.SilkS")
-        (effects (font (size 0.7 0.7) (thickness 0.1)))
+    (fp_text value "VIN Scaled" (at 3.75 -3.75 45) (layer "F.SilkS")
+        (effects (font (size 1 1) (thickness 0.15)))
     )
     (fp_text user "${REFERENCE}" (at 0 -2) (layer "F.Fab")
@@
   )
   (footprint "Package_TO_SOT_SMD:TO-263-2" locked (layer "F.Cu")
-    (at 184 108.375 90)
+    (at 185 108.375 90)
     (descr "TO-263 / D2PAK / DDPAK SMD package, http://www.infineon.com/cms/en/product/packages/PG-TO263/PG-TO263-3-1/")
     (tags "D2PAK DDPAK TO-263 D2PAK-3 TO-263-3 SOT-404")
@@
         (effects (font (size 1 1) (thickness 0.15)))
     )
-    (fp_text value "Telemetry" (at 1.75 2.8 270) (layer "F.SilkS")
-        (effects (font (size 0.7 0.7) (thickness 0.1)))
+    (fp_text value "Telemetry" (at 2 6.3 270) (layer "F.SilkS")
+        (effects (font (size 1 1) (thickness 0.15) bold))
     )
     (fp_text user "${REFERENCE}" (at 0 3.81 270) (layer "F.Fab") hide
@@
         (effects (font (size 1 1) (thickness 0.15)))
     )
-    (fp_text value "Gate Log" (at -2.75 2.75 45) (layer "F.SilkS")
-        (effects (font (size 0.7 0.7) (thickness 0.1)))
+    (fp_text value "Gate Log" (at 1.5 1.5 45) (layer "F.SilkS")
+        (effects (font (size 1 1) (thickness 0.15)))
     )
     (fp_text user "${REFERENCE}" (at 0 -2) (layer "F.Fab")
@@
   (gr_line locked (start 160 144) (end 160 91)
     (stroke (width 0.15) (type dash_dot)) (layer "Dwgs.User"))
-  (gr_line locked (start 184 144) (end 184 91)
+  (gr_line locked (start 185 144) (end 185 91)
     (stroke (width 0.15) (type dash_dot)) (layer "Dwgs.User"))
-  (gr_line locked (start 136 144) (end 136 91)
+  (gr_line locked (start 135 144) (end 135 91)
     (stroke (width 0.15) (type dash_dot)) (layer "Dwgs.User"))
   (gr_line locked (start 110 90) (end 110 145)
@@
   )
   (dimension locked (type aligned) (layer "Dwgs.User")
-    (pts (xy 110 145.000001) (xy 136 145))
+    (pts (xy 110 145.000001) (xy 135 145))
     (height 3.999999)
-    (gr_text "26,0000  mm" (at 123 147.85) (layer "Dwgs.User")
+    (gr_text "25,0000  mm" (at 122.5 147.85) (layer "Dwgs.User")
       (effects (font (size 1 1) (thickness 0.15)))
     )
@@
   )
   (dimension locked (type aligned) (layer "Dwgs.User")
-    (pts (xy 184 145.000001) (xy 210 145))
+    (pts (xy 185 145.000001) (xy 210 145))
     (height 3.999999)
-    (gr_text "26,0000  mm" (at 197 147.85) (layer "Dwgs.User")
+    (gr_text "25,0000  mm" (at 197.5 147.85) (layer "Dwgs.User")
       (effects (font (size 1 1) (thickness 0.15)))
     )
@@
   (via (at 121 92) (size 1.2) (drill 1) (layers "F.Cu" "B.Cu") (free) (net 24))
   (via (at 157 95) (size 1.2) (drill 1) (layers "F.Cu" "B.Cu") (free) (net 24))
+  (via (at 142 101) (size 1.2) (drill 1) (layers "F.Cu" "B.Cu") (free) (net 24))
   (via (at 112 92) (size 1.2) (drill 1) (layers "F.Cu" "B.Cu") (free) (net 24))
   (via (at 157 104) (size 1.2) (drill 1) (layers "F.Cu" "B.Cu") (free) (net 24))
@@
   (via (at 139 92) (size 1.2) (drill 1) (layers "F.Cu" "B.Cu") (free) (net 24))
   (via (at 142 95) (size 1.2) (drill 1) (layers "F.Cu" "B.Cu") (free) (net 24))
+  (via (at 142 104) (size 1.2) (drill 1) (layers "F.Cu" "B.Cu") (free) (net 24))
   (via (at 151 98) (size 1.2) (drill 1) (layers "F.Cu" "B.Cu") (free) (net 24))
   (via (at 115 95) (size 1.2) (drill 1) (layers "F.Cu" "B.Cu") (free) (net 24))
@@
   (via (at 118 104) (size 1.2) (drill 1) (layers "F.Cu" "B.Cu") (free) (net 24))
   (via (at 148 104) (size 1.2) (drill 1) (layers "F.Cu" "B.Cu") (free) (net 24))
+  (via (at 142 107) (size 1.2) (drill 1) (layers "F.Cu" "B.Cu") (free) (net 24))
   (via (at 124 95) (size 1.2) (drill 1) (layers "F.Cu" "B.Cu") (free) (net 24))
   (via (at 148 95) (size 1.2) (drill 1) (layers "F.Cu" "B.Cu") (free) (net 24))
@@
   (via (at 196 95) (size 1.2) (drill 1) (layers "F.Cu" "B.Cu") (free) (net 26))
   (via (at 184 98) (size 1.2) (drill 1) (layers "F.Cu" "B.Cu") (free) (net 26))
+  (via (at 178 104) (size 1.2) (drill 1) (layers "F.Cu" "B.Cu") (free) (net 26))
   (via (at 172 98) (size 1.2) (drill 1) (layers "F.Cu" "B.Cu") (free) (net 26))
   (via (at 163 92) (size 1.2) (drill 1) (layers "F.Cu" "B.Cu") (free) (net 26))
@@
   (via (at 202 92) (size 1.2) (drill 1) (layers "F.Cu" "B.Cu") (free) (net 26))
   (via (at 175 104) (size 1.2) (drill 1) (layers "F.Cu" "B.Cu") (free) (net 26))
+  (via (at 178 101) (size 1.2) (drill 1) (layers "F.Cu" "B.Cu") (free) (net 26))
   (via (at 187 95) (size 1.2) (drill 1) (layers "F.Cu" "B.Cu") (free) (net 26))
   (via (at 166 104) (size 1.2) (drill 1) (layers "F.Cu" "B.Cu") (free) (net 26))
@@
     (polygon
       (pts
-        (xy 135.5 117.5)
+        (xy 134.5 117.5)
         (xy 110 117.5)
         (xy 110 110)
-        (xy 135.5 110)
+        (xy 134.5 110)
       )
     )
@@
       (pts
         (xy 200.5 116.5)
-        (xy 183.5 116.5)
-        (xy 183.5 111)
+        (xy 185.5 116.5)
+        (xy 185.5 111)
         (xy 200.5 111)
       )
@@
     (polygon
       (pts
-        (xy 182.5 116.5)
+        (xy 184.5 116.5)
         (xy 179 116.5)
         (xy 179 111)
-        (xy 182.5 111)
+        (xy 184.5 111)
       )
     )
@@
       (pts
         (xy 142 116.5)
-        (xy 136.5 116.5)
-        (xy 136.5 111)
+        (xy 136 116.5)
+        (xy 136 111)
         (xy 142 111)
       )
